File: mcu.kicad_sch (KiCad schematic)
At the start: 0 parts

Commit message: Ajouter des composants + connexion page "MCU"
Parts:
- added C301: 10u, symbol Device:C
- added C302, C304, C305: 100n, symbol Device:C
- added C303: 1u, symbol Device:C
- added D301: A-SP194BR5C-C01-3T, LED_SMD:LED_0603_1608Metric, symbol Device:LED
- added Q301, Q302: L8050QLT1G, Package_TO_SOT_SMD:SOT-23, symbol tuto-kicad-temp-logger:L8050QLT1G
- added R301, R306, R307: 10k, symbol Device:R
- added R302, R303: 4.7k, symbol Device:R
- added R304: 47k, symbol Device:R
- added R305: 270R, symbol Device:R
- added SW301, SW302: TE_FSM4JSMATR, tuto-kicad-temp-logger:TE_FSM4JSMATR, symbol tuto-kicad-temp-logger:TE_FSM4JSMATR
- added TP301, TP302, TP303, TP304, TP305: TestPoint, symbol Connector:TestPoint
- added U301: ESP32-C3-WROOM-02, PCM_Espressif:ESP32-C3-WROOM-02, symbol PCM_Espressif:ESP32-C3-WROOM-02
Connections:
- new net: TP302.1, U301.13 (GPIO18/USB_D-)
- new net: TP303.1, U301.14 (GPIO19/USB_D+)
- new net: Q302.1 (B), R307.2
- new net: D301.2 (A), R305.2
- new net: Q301.1 (B), R306.2
- new net +3V3: C301.1, C302.1, R301.1, R302.1, R303.1, R304.1, U301.1 (3V3)
- new net CHIP_PU: C303.1, C304.2, Q301.3 (C), R301.2, SW301.3 (K), SW301.4 (A), TP301.1, U301.2 (EN/CHIP_PU)
- new net DTR: Q302.2 (E), R306.1
- new net GND: C301.2, C302.2, C303.2, C304.1, C305.1, D301.1 (K), SW301.1, SW301.2, SW302.1, SW302.2, U301.19 (GND), U301.9 (GND)
- new net GPIO10: R305.1, TP305.1, U301.10 (GPIO10)
- new net GPIO9: C305.2, Q302.3 (C), SW302.3 (K), SW302.4 (A), TP304.1, U301.8 (GPIO9)
- new net I2C.SCL: R302.2, U301.6 (GPIO7)
- new net I2C.SDA: R303.2, U301.7 (GPIO8)
- new net RTS: Q301.2 (E), R307.1
- new net SD.CD: U301.5 (GPIO6)
- new net SD.CS: U301.4 (GPIO5/ADC2_CH0)
- new net SD.MISO: U301.15 (GPIO3/ADC1_CH3)
- new net SD.MOSI: U301.3 (GPIO4/ADC1_CH4)
- new net SD.SCK: R304.2, U301.16 (GPIO2/ADC1_CH2)
- new net UART.ESP32_RX: U301.11 (GPIO20/U0RXD)
- new net UART.ESP32_TX: U301.12 (GPIO21/U0TXD)
- no-connect marks 0 -> 2

Commit message: Vérification des règles électriques
Parts:
- C301, C302, C303, C304, C305: footprint (none) -> Capacitor_SMD:C_0402_1005Metric
- R301, R302, R303, R304, R305, R306, R307: footprint (none) -> Resistor_SMD:R_0402_1005Metric
- TP301, TP302, TP303, TP304, TP305: footprint (none) -> TestPoint:TestPoint_Pad_D2.0mm
Changed lines of the file:
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@@
 			)
 		)
-		(property "Footprint" ""
+		(property "Footprint" "Capacitor_SMD:C_0402_1005Metric"
 			(at 125.4252 36.83 0)
 			(effects
@@
 			)
 		)
-		(property "Footprint" ""
+		(property "Footprint" "TestPoint:TestPoint_Pad_D2.0mm"
 			(at 172.72 60.96 0)
 			(effects
@@
 			)
 		)
-		(property "Footprint" ""
+		(property "Footprint" "TestPoint:TestPoint_Pad_D2.0mm"
 			(at 172.72 63.5 0)
 			(effects
@@
 			)
 		)
-		(property "Footprint" ""
+		(property "Footprint" "Resistor_SMD:R_0402_1005Metric"
 			(at 205.232 69.85 90)
 			(effects
@@
 			)
 		)
-		(property "Footprint" ""
+		(property "Footprint" "Capacitor_SMD:C_0402_1005Metric"
 			(at 113.9952 36.83 0)
 			(effects
@@
 			)
 		)
-		(property "Footprint" ""
+		(property "Footprint" "Capacitor_SMD:C_0402_1005Metric"
 			(at 210.82 138.7348 0)
 			(effects
@@
 			)
 		)
-		(property "Footprint" ""
+		(property "Footprint" "Resistor_SMD:R_0402_1005Metric"
 			(at 58.42 159.258 90)
 			(effects
@@
 			)
 		)
-		(property "Footprint" ""
+		(property "Footprint" "Capacitor_SMD:C_0402_1005Metric"
 			(at 87.3252 57.15 0)
 			(effects
@@
 			)
 		)
-		(property "Footprint" ""
+		(property "Footprint" "Resistor_SMD:R_0402_1005Metric"
 			(at 247.142 127 90)
 			(effects
@@
 			)
 		)
-		(property "Footprint" ""
+		(property "Footprint" "TestPoint:TestPoint_Pad_D2.0mm"
 			(at 171.45 88.9 0)
 			(effects
@@
 			)
 		)
-		(property "Footprint" ""
+		(property "Footprint" "Resistor_SMD:R_0402_1005Metric"
 			(at 205.232 93.98 90)
 			(effects
@@
 			)
 		)
-		(property "Footprint" ""
+		(property "Footprint" "Resistor_SMD:R_0402_1005Metric"
 			(at 197.612 69.85 90)
 			(effects
@@
 			)
 		)
-		(property "Footprint" ""
+		(property "Footprint" "Resistor_SMD:R_0402_1005Metric"
 			(at 58.42 138.938 90)
 			(effects
@@
 			)
 		)
-		(property "Footprint" ""
+		(property "Footprint" "TestPoint:TestPoint_Pad_D2.0mm"
 			(at 171.45 86.36 0)
 			(effects
@@
 			)
 		)
-		(property "Footprint" ""
+		(property "Footprint" "Capacitor_SMD:C_0402_1005Metric"
 			(at 176.53 138.7348 0)
 			(effects
@@
 			)
 		)
-		(property "Footprint" ""
+		(property "Footprint" "Resistor_SMD:R_0402_1005Metric"
 			(at 84.582 41.91 90)
 			(effects
@@
 			)
 		)
-		(property "Footprint" ""
+		(property "Footprint" "TestPoint:TestPoint_Pad_D2.0mm"
 			(at 86.36 53.34 0)
 			(effects
