File: usb_power_supply.kicad_sch (KiCad schematic)
At the start: 0 parts

Commit message: Ajout des composants et connexion page "USB + Power supply"
Parts:
- added C201, C204, C205: 10u, symbol Device:C
- added C202, C203: 100n, symbol Device:C
- added C206: 1u, symbol Device:C
- added D201, D202, D203: LESD5D5.0CT1G, tuto-kicad-temp-logger:D_SOD-523_non-pol, symbol tuto-kicad-temp-logger:LESD5D5.0CT1G
- added D204: A-SP194BR5C-C01-3T, LED_SMD:LED_0603_1608Metric, symbol Device:LED
- added J201: HOOYA_USB_306F, tuto-kicad-temp-logger:HOOYA_USB_306F, symbol tuto-kicad-temp-logger:HOOYA_USB_306F
- added J202: Conn_01x01_Pin, symbol Connector:Conn_01x01_Pin
- added R201: 270R, symbol Device:R
- added R202, R203: 5k1, symbol Device:R
- added R204: 1k, symbol Device:R
- added R205: 22.1k 1%, symbol Device:R
- added R206: 47.1k 1%, symbol Device:R
- added TP201, TP202, TP203, TP204, TP205, TP206, TP207: TestPoint, symbol Connector:TestPoint
- added U201: SGM2212-3.3XKC3G, Package_TO_SOT_SMD:SOT-223, symbol tuto-kicad-temp-logger:SGM2212-3.3XKC3G
- added U202: CP2102N-Axx-xQFN28, Package_DFN_QFN:QFN-28-1EP_5x5mm_P0.5mm_EP3.35x3.35mm, symbol Interface_USB:CP2102N-Axx-xQFN28
Connections:
- new net: D204.2 (A), R201.2
- new net: R204.2, U202.9 (~{RST})
- new net: C206.1, R205.2, R206.1, U202.8 (VBUS)
- new net +3V3: C203.1, C204.1, C205.1, R201.1, R204.1, TP202.1, U201.2 (VOUT), U201.4 (VOUT_PAD), U202.6 (VDD), U202.7 (VREGIN)
- new net CC1: J201.A5 (CC1), R203.1
- new net CC2: J201.B5 (CC2), R202.1
- new net DTR: TP206.1, U202.28 (~{DTR})
- new net GND: C201.2, C202.2, C203.2, C204.2, C205.2, C206.2, D201.1 (A1), D202.1 (A1), D203.1 (A1), D204.1 (K), J201.A1 (GND), J201.A12 (GND), J201.B1 (GND), J201.B12 (GND), J201.SH (SHIELD), J202.1 (Pin_1), R202.2, R203.2, R206.2, TP207.1, U201.1 (GND), U202.29 (GND), U202.3 (GND)
- new net RTS: TP205.1, U202.24 (~{RTS})
- new net UART.ESP32_RX: TP203.1, U202.26 (TXD)
- new net UART.ESP32_TX: TP204.1, U202.25 (RXD)
- new net USB_DATA.DN: D203.2 (A2), J201.A7 (DN1), J201.B7 (DN2), U202.5 (D-)
- new net USB_DATA.DP: D202.2 (A2), J201.A6 (DP1), J201.B6 (DP2), U202.4 (D+)
- new net VBUS: C201.1, C202.1, D201.2 (A2), J201.A4 (VBUS), J201.A9 (VBUS), J201.B4 (VBUS), J201.B9 (VBUS), R205.1, TP201.1, U201.3 (VIN)
- no-connect marks 0 -> 26

Commit message: Vérification des règles électriques
Parts:
- C201, C202, C203, C204, C205, C206: footprint (none) -> Capacitor_SMD:C_0402_1005Metric
- J202: footprint (none) -> Connector_PinHeader_2.54mm:PinHeader_1x01_P2.54mm_Vertical
- R201, R202, R203, R204, R205, R206: footprint (none) -> Resistor_SMD:R_0402_1005Metric
- TP201, TP202, TP203, TP204, TP205, TP206, TP207: footprint (none) -> TestPoint:TestPoint_Pad_D2.0mm
Changed lines of the file:
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@@
 			)
 		)
-		(property "Footprint" ""
+		(property "Footprint" "Resistor_SMD:R_0402_1005Metric"
 			(at 243.332 68.58 90)
 			(effects
@@
 			)
 		)
-		(property "Footprint" ""
+		(property "Footprint" "Capacitor_SMD:C_0402_1005Metric"
 			(at 166.0652 71.12 0)
 			(effects
@@
 			)
 		)
-		(property "Footprint" ""
+		(property "Footprint" "Capacitor_SMD:C_0402_1005Metric"
 			(at 230.8352 71.12 0)
 			(effects
@@
 			)
 		)
-		(property "Footprint" ""
+		(property "Footprint" "TestPoint:TestPoint_Pad_D2.0mm"
 			(at 240.03 153.67 0)
 			(effects
@@
 			)
 		)
-		(property "Footprint" ""
+		(property "Footprint" "TestPoint:TestPoint_Pad_D2.0mm"
 			(at 181.61 62.23 0)
 			(effects
@@
 			)
 		)
-		(property "Footprint" ""
+		(property "Footprint" "Capacitor_SMD:C_0402_1005Metric"
 			(at 218.1352 71.12 0)
 			(effects
@@
 			)
 		)
-		(property "Footprint" ""
+		(property "Footprint" "Resistor_SMD:R_0402_1005Metric"
 			(at 68.072 119.38 90)
 			(effects
@@
 			)
 		)
-		(property "Footprint" ""
+		(property "Footprint" "Resistor_SMD:R_0402_1005Metric"
 			(at 24.892 91.44 90)
 			(effects
@@
 			)
 		)
-		(property "Footprint" ""
+		(property "Footprint" "Capacitor_SMD:C_0402_1005Metric"
 			(at 26.3652 134.62 0)
 			(effects
@@
 			)
 		)
-		(property "Footprint" ""
+		(property "Footprint" "TestPoint:TestPoint_Pad_D2.0mm"
 			(at 130.81 125.73 0)
 			(effects
@@
 			)
 		)
-		(property "Footprint" ""
+		(property "Footprint" "Capacitor_SMD:C_0402_1005Metric"
 			(at 82.2452 116.84 0)
 			(effects
@@
 			)
 		)
-		(property "Footprint" ""
+		(property "Footprint" "TestPoint:TestPoint_Pad_D2.0mm"
 			(at 222.25 62.23 0)
 			(effects
@@
 			)
 		)
-		(property "Footprint" ""
+		(property "Footprint" "Resistor_SMD:R_0402_1005Metric"
 			(at 84.582 91.44 90)
 			(effects
@@
 			)
 		)
-		(property "Footprint" ""
+		(property "Footprint" "Resistor_SMD:R_0402_1005Metric"
 			(at 33.782 130.81 90)
 			(effects
@@
 			)
 		)
-		(property "Footprint" ""
+		(property "Footprint" "TestPoint:TestPoint_Pad_D2.0mm"
 			(at 130.81 128.27 0)
 			(effects
@@
 			)
 		)
-		(property "Footprint" ""
+		(property "Footprint" "Resistor_SMD:R_0402_1005Metric"
 			(at 33.782 123.19 90)
 			(effects
@@
 			)
 		)
-		(property "Footprint" ""
+		(property "Footprint" "TestPoint:TestPoint_Pad_D2.0mm"
 			(at 120.65 130.81 0)
 			(effects
@@
 			)
 		)
-		(property "Footprint" ""
+		(property "Footprint" "Connector_PinHeader_2.54mm:PinHeader_1x01_P2.54mm_Vertical"
 			(at 240.03 154.94 0)
 			(effects
@@
 			)
 		)
-		(property "Footprint" ""
+		(property "Footprint" "Capacitor_SMD:C_0402_1005Metric"
 			(at 177.4952 71.12 0)
 			(effects
@@
 			)
 		)
-		(property "Footprint" ""
+		(property "Footprint" "TestPoint:TestPoint_Pad_D2.0mm"
 			(at 120.65 138.43 0)
 			(effects
